File: pcb/revA/audio.kicad_sch (KiCad schematic)
At the start: 43 parts, among them J3 PJ307, J4 Conn_01x04, U1 YMF262-M, U15 SAM2695, U16 PCM1808PWR, U25 PCM5102A

Commit message: Initial firmware
Parts:
- renumbered C67 to C16, C68 to C17, C69 to C18, C70 to C19, C71 to C20, C72 to C21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
Other:
- note added: "SOUND OUT"
- note removed: "SOUND"
- title: karabas-Megasound -> Karabas-MegaBuzz
- moved on the sheet: C16, C17, C18, C19, C20, C21, C22, C23, C24, C25, C26, C27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
