File: pcb/revA/fpga1.kicad_sch (KiCad schematic)
At the start: 14 parts, among them U7 XC6SLX25-FTG256

Commit message: Initial firmware
Parts:
- added TP1, TP2, TP3, TP4, TP5, TP6, TP7: TestPoint, TestPoint:TestPoint_Pad_D1.5mm, symbol Connector:TestPoint
- renumbered C27 to C1, C36 to C10, C37 to C11, C38 to C12, C39 to C13, C28 to C2, C29 to C3, C30 to C4, C31 to C5, C32 to C6, C33 to C7, C34 to C8, C35 to C9, U7 to U1
Connections:
- net at U1.A11 (IO_L39N_0): now also TP2.1
- net at U1.A12 (IO_L62N_VREF_0): now also TP1.1
- net ~{BTN_RST}: now reaches U1.A13 (IO_L63N_SCP6_0)
- net at U1.B12 (IO_L62P_0): now also TP3.1
- net at U1.C13 (IO_L63P_SCP7_0): now also TP4.1
- net at U1.F13 (IO_L32P_A17_M1A8_1): now also TP6.1
- net at U1.F14 (IO_L32N_A16_M1A9_1): now also TP7.1
- net at U1.G12 (IO_L38P_A5_M1CLK_1): now also TP5.1
- no-connect marks 0 -> 40
Other:
- title: karabas-Megasound -> Karabas-MegaBuzz
