File: pcb/revA/fpga2.kicad_sch (KiCad schematic)
At the start: 11 parts, among them J6 FPGA JTAG, U12 W25Q128JVS, U7 XC6SLX25-FTG256, X2 50 MHz

Commit message: Initial firmware
Parts:
- added TP10, TP11, TP12, TP13, TP14, TP15, TP16, TP17, TP18, TP8, TP9: TestPoint, TestPoint:TestPoint_Pad_D1.5mm, symbol Connector:TestPoint
- renumbered C40 to C14, C75 to C15, J6 to J1, R15 to R1, R10 to R2, R17 to R3, R18 to R4, U7 to U1, U12 to U2, X2 to X1
Connections:
- net VCC3_3 is gone; now on net +3V3: U1.T11 (IO_L1N_M0_CMPMISO_2)
- net CONF_CLK: now also TP13.1
- net CONF_DONE: now also TP10.1
- net CONF_INIT_B: now also TP9.1
- net CONF_IO0: now also TP14.1
- net CONF_IO1: now also TP15.1
- net CONF_IO2: now also TP16.1
- net CONF_IO3: now also TP17.1
- net CONF_M1: now also TP18.1
- net CONF_PRG_B: now also TP11.1
- net ~{CONF_CS}: now also TP12.1
- net ~{xRST}: now reaches U1.L5 (IO_L45N_M3ODT_3)
- net at U1.M12 (IO_L2P_CMPCLK_2): now also TP8.1
- no-connect marks 4 -> 27
Other:
- note added: "CONF FLASH"
- note added: "MASTER CLOCK"
- note removed: "Master Clock"
- title: karabas-Megasound -> Karabas-MegaBuzz
- moved on the sheet: C15, JP1, R2, R4, U2
