File: pcb/revA/interfaces.kicad_sch (KiCad schematic)
At the start: 15 parts, among them J2 Conn_02x30_Row_Letter_First, SW1 SW_DIP_x05, U10 SN74CB3T3245PW, U2 74AHCT1G125DB, U4 SN74CB3T3245PW, U8 SN74CB3T3245PW, U9 SN74CB3T3245PW

Commit message: Initial firmware
Parts:
- added BTN1: Reset, footprints:SW_SPST_PTS810_handsoldering, symbol Switch:SW_Push
- added R46: 10k, Resistor_SMD:R_0603_1608Metric_Pad0.98x0.95mm_HandSolder, symbol Device:R
- added U22: SN74LV1T34DBV, Package_TO_SOT_SMD:SOT-23-5_HandSoldering, symbol Logic_LevelTranslator:SN74LV1T34DBV
- renumbered R1 to R10, R4 to R11, R6 to R12, R16 to R5, R19 to R6, R37 to R7, R38 to R8, R39 to R9, U2 to U3, U9 to U5, U8 to U6, U10 to U7
Connections:
- net +3V3: now also R46.1, U22.5 (VCC)
- net GND: now also BTN1.2, U22.3 (GND)
- net ~{RST}: now also U22.2 (A)
- new net ~{BTN_RST}: BTN1.1, R46.2
- new net ~{xRST}: U22.4 (Y)
Other:
- note added: "LEVEL SHIFTERS"
- note added: "RESET BUTTON"
- title: karabas-Megasound -> Karabas-MegaBuzz
- moved on the sheet: J2, R10, R11, R12, R5, R6, R7, R8, R9, SW1, U3, U4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
