File: pcb/revA/karabas-megasound.kicad_pcb (KiCad board)
At the start: 4 copper layers, 92.2 x 44 mm, 157 parts, among them J2 Conn_02x30_Row_Letter_First, J3 PJ307, J4 Conn_01x04, J5 5V_PRG, J6 FPGA JTAG, SW1 SW_DIP_x05, U1 YMF262-M, U10 SN74CB3T3245PW, U11 1117-1.2, U12 W25Q128JVS, U15 SAM2695, U16 PCM1808PWR, U2 74AHCT1G125DB, U25 PCM5102A, U3 CY62167EV30LL, U4 SN74CB3T3245PW, U5 1117-3.3, U6 1117-3.3, U7 XC6SLX25-FTG256, U8 SN74CB3T3245PW, U9 SN74CB3T3245PW, X2 50 MHz

Commit message: Initial firmware
Parts:
- removed LOGO1: graphic, footprints:opl3
- added BTN1: RESET, footprints:SW_SPST_PTS810_handsoldering, F.Cu at (172.1, 94.9)
- added R46: 10k, Resistor_SMD:R_0603_1608Metric_Pad0.98x0.95mm_HandSolder, B.Cu at (172.1, 94.9)
- added TP1: TestPoint, TestPoint:TestPoint_Pad_D1.5mm, B.Cu at (177.1, 98.2)
- added TP10: TestPoint, TestPoint:TestPoint_Pad_D1.5mm, B.Cu at (172.0, 115.4)
- added TP11: TestPoint, TestPoint:TestPoint_Pad_D1.5mm, B.Cu at (157.5, 121.0)
- added TP12: TestPoint, TestPoint:TestPoint_Pad_D1.5mm, B.Cu at (179.2, 119.6)
- added TP13: TestPoint, TestPoint:TestPoint_Pad_D1.5mm, B.Cu at (170.8, 121.4)
- added TP14: TestPoint, TestPoint:TestPoint_Pad_D1.5mm, B.Cu at (171.8, 123.9)
- added TP15: TestPoint, TestPoint:TestPoint_Pad_D1.5mm, B.Cu at (175.1, 119.6)
- added TP16: TestPoint, TestPoint:TestPoint_Pad_D1.5mm, B.Cu at (172.6, 119.6)
- added TP17: TestPoint, TestPoint:TestPoint_Pad_D1.5mm, B.Cu at (174.4, 123.9)
- added TP18: TestPoint, TestPoint:TestPoint_Pad_D1.5mm, B.Cu at (175.5, 115.4)
- added TP2: TestPoint, TestPoint:TestPoint_Pad_D1.5mm, B.Cu at (177.1, 100.8)
- added TP3: TestPoint, TestPoint:TestPoint_Pad_D1.5mm, B.Cu at (177.1, 103.3)
- added TP4: TestPoint, TestPoint:TestPoint_Pad_D1.5mm, B.Cu at (177.1, 105.8)
- added TP5: TestPoint, TestPoint:TestPoint_Pad_D1.5mm, B.Cu at (183.1, 98.2)
- added TP6: TestPoint, TestPoint:TestPoint_Pad_D1.5mm, B.Cu at (183.1, 100.8)
- added TP7: TestPoint, TestPoint:TestPoint_Pad_D1.5mm, B.Cu at (183.1, 103.3)
- added TP8: TestPoint, TestPoint:TestPoint_Pad_D1.5mm, B.Cu at (183.1, 105.8)
- added TP9: TestPoint, TestPoint:TestPoint_Pad_D1.5mm, B.Cu at (161.0, 121.0)
- added U22: SN74LV1T34DBV, Package_TO_SOT_SMD:SOT-23-5_HandSoldering, B.Cu at (150.5, 104.1)
- J5: value 5V_PRG -> 5VP
- moved J5 32.5 mm to (181.1, 125.0), turned to 90 degrees
- moved LOGO2 1.08 mm to (116.6, 119.9)
- moved C29 0.31 mm to (127.8, 102.8)
- renumbered C27 to C1, C36 to C10, C37 to C11, C38 to C12, C39 to C13, C40 to C14, C75 to C15, C67 to C16, C68 to C17, C69 to C18, C70 to C19, C28 to C2, C71 to C20, C72 to C21, C73 to C22, C74 to C23, C63 to C24, C62 to C25, C64 to C26, C102 to C27, C95 to C28, C65 to C29, C29 to C3, C66 to C30, C103 to C31, C97 to C32, C96 to C33, C86 to C34, C99 to C35, C98 to C36, C101 to C37, C100 to C38, C45 to C39, C30 to C4, C11 to C40, C21 to C41, C7 to C42, C12 to C43, C22 to C44, C13 to C45, C14 to C46, C8 to C47, C15 to C48, C26 to C49, C31 to C5, C9 to C50, C10 to C51, C41 to C52, C42 to C53, C43 to C54, C44 to C55, C32 to C6, C33 to C7, C34 to C8, C35 to C9, D2 to D1, D11 to D10, D12 to D11, D13 to D12, D14 to D13, D15 to D14, D16 to D15, D17 to D16, D3 to D2, D4 to D3, D5 to D4, D6 to D5, D7 to D6, D8 to D7, D9 to D8, D10 to D9, J6 to J1, R15 to R1, R1 to R10, R4 to R11, R6 to R12, R61 to R13, R62 to R14, R65 to R15, R66 to R16, R45 to R17, R46 to R18, R43 to R19, R10 to R2, R44 to R20, R60 to R21, R59 to R22, R63 to R23, R64 to R24, R57 to R25, R58 to R26, R12 to R27, R13 to R28, R14 to R29, R17 to R3, R21 to R30, R22 to R31, R23 to R32, R24 to R33, R25 to R34, R26 to R35, R27 to R36, R28 to R37, R29 to R38, R30 to R39, R18 to R4, R31 to R40, R32 to R41, R33 to R42, R34 to R43, R35 to R44, R36 to R45, R16 to R5, R19 to R6, R37 to R7, R38 to R8, R39 to R9, U7 to U1, U25 to U10, U16 to U11, U3 to U12, U5 to U13, U6 to U14, U11 to U15, U12 to U2, U2 to U3, U9 to U5, U8 to U6, U10 to U7, U1 to U8, U15 to U9, X2 to X1
Connections:
- U1 pad A11: unconnected-(U7A-IO_L39N_0-PadA11) -> Net-(U1A-IO_L39N_0)
- U1 pad A12: unconnected-(U7A-IO_L62N_VREF_0-PadA12) -> Net-(U1A-IO_L62N_VREF_0)
- U1 pad A13: unconnected-(U7A-IO_L63N_SCP6_0-PadA13) -> ~{BTN_RST}
- U1 pad B12: unconnected-(U7A-IO_L62P_0-PadB12) -> Net-(U1A-IO_L62P_0)
- U1 pad C13: unconnected-(U7A-IO_L63P_SCP7_0-PadC13) -> Net-(U1A-IO_L63P_SCP7_0)
- U1 pad F13: unconnected-(U7A-IO_L32P_A17_M1A8_1-PadF13) -> Net-(U1A-IO_L32P_A17_M1A8_1)
- U1 pad F14: unconnected-(U7A-IO_L32N_A16_M1A9_1-PadF14) -> Net-(U1A-IO_L32N_A16_M1A9_1)
- U1 pad G12: unconnected-(U7A-IO_L38P_A5_M1CLK_1-PadG12) -> Net-(U1A-IO_L38P_A5_M1CLK_1)
- U1 pad L5: unconnected-(U7B-IO_L45N_M3ODT_3-PadL5) -> ~{xRST}
- U1 pad M12: unconnected-(U7B-IO_L2P_CMPCLK_2-PadM12) -> Net-(U1B-IO_L2P_CMPCLK_2)
- U1 pad T11: VCC3_3 -> +3V3
Routing:
- net Net-(U1A-IO_L38P_A5_M1CLK_1): track 0.00 -> 23.2 mm, vias 0 -> 1
- net ~{xRST}: track 0.00 -> 21.7 mm, vias 0 -> 2
- net Net-(U1A-IO_L32P_A17_M1A8_1): track 0.00 -> 19.8 mm, vias 0 -> 1
- net Net-(U1B-IO_L2P_CMPCLK_2): track 0.00 -> 17.5 mm, vias 0 -> 1
- net Net-(U1A-IO_L32N_A16_M1A9_1): track 0.00 -> 16.7 mm, vias 0 -> 1
- net +3V3: track 157.5 -> 169.8 mm, vias 46 -> 47
- net Net-(U1A-IO_L39N_0): track 0.00 -> 11.5 mm, vias 0 -> 1
- net Net-(U1A-IO_L63P_SCP7_0): track 0.00 -> 11.4 mm, vias 0 -> 1
- net Net-(U1A-IO_L62N_VREF_0): track 0.00 -> 11.1 mm, vias 0 -> 1
- net ~{BTN_RST}: track 0.00 -> 10.9 mm, vias 0 -> 2
- net CONF_INIT_B: track 0.00 -> 10.1 mm, vias 0 -> 2
- net +5V: track 182.3 -> 172.3 mm, vias 19 -> 18
- net Net-(U1A-IO_L62P_0): track 0.00 -> 9.84 mm, vias 0 -> 1
- net CONF_PRG_B: track 2.15 -> 9.08 mm, vias 1 -> 2
- net CONF_DONE: track 0.00 -> 3.34 mm, vias 0 -> 1
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Other:
- board text added: "${TITLE}"
- board text added: "+"
- board text added: "GND"
- board text added: "L"
- board text added: "R"
- board text removed: "Karabas Megasound"
- board text removed: "ZX Spectrum Soundcard General Sound Turbo-Sound FM OPL3 MIDI SAA1099 Soundrive Covox Beeper"
