File: pcb/revA/memory.kicad_sch (KiCad schematic)
At the start: 2 parts, among them U3 CY62167EV30LL

Commit message: Initial firmware
Parts:
- renumbered C45 to C39, U3 to U12
Other:
- note added: "GS RAM"
- title: karabas-Megasound -> Karabas-MegaBuzz
Changed lines of the file:
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@@
 	(paper "A4")
 	(title_block
-		(title "karabas-Megasound")
-		(date "2026-04-02")
-		(rev "B")
+		(title "Karabas-MegaBuzz")
+		(date "2026-04-18")
+		(rev "A")
 		(company "Andy Karpov")
+	)
+	(rectangle
+		(start 30.48 24.765)
+		(end 93.98 114.3)
+		(stroke
+			(width 0)
+			(type dash)
+		)
+		(fill
+			(type none)
+		)
+	)
+	(text "GS RAM"
+		(exclude_from_sim no)
+		(at 30.48 24.13 0)
+		(effects
+			(font
+				(size 2 2)
+				(thickness 0.4)
+				(bold yes)
+				(italic yes)
+			)
+			(justify left bottom)
+		)
 	)
 	(junction
@@
 		(in_pos_files yes)
 		(dnp no)
-		(property "Reference" "C45"
+		(property "Reference" "C39"
 			(at 87.6808 93.98 90)
 			(show_name no)
@@
 			(project "karabas-megasound"
 				(path "/eff1afb7-47ba-46af-a815-4a07fb8d674b/1ef77d13-3c60-4080-9817-a45398794587"
-					(reference "C45")
+					(reference "C39")
 					(unit 1)
 				)
@@
 		(in_pos_files yes)
 		(dnp no)
-		(property "Reference" "#PWR084"
+		(property "Reference" "#PWR0105"
 			(at 80.01 100.33 0)
 			(hide yes)
@@
 			(project "karabas-megasound"
 				(path "/eff1afb7-47ba-46af-a815-4a07fb8d674b/1ef77d13-3c60-4080-9817-a45398794587"
-					(reference "#PWR084")
+					(reference "#PWR0105")
 					(unit 1)
 				)
@@
 		(in_pos_files yes)
 		(dnp no)
-		(property "Reference" "#PWR028"
+		(property "Reference" "#PWR0101"
 			(at 38.1 102.87 0)
 			(hide yes)
@@
 			(project "karabas-megasound"
 				(path "/eff1afb7-47ba-46af-a815-4a07fb8d674b/1ef77d13-3c60-4080-9817-a45398794587"
-					(reference "#PWR028")
+					(reference "#PWR0101")
 					(unit 1)
 				)
@@
 		(in_pos_files yes)
 		(dnp no)
-		(property "Reference" "#PWR027"
+		(property "Reference" "#PWR0100"
 			(at 38.1 90.17 0)
 			(hide yes)
@@
 			(project "karabas-megasound"
 				(path "/eff1afb7-47ba-46af-a815-4a07fb8d674b/1ef77d13-3c60-4080-9817-a45398794587"
-					(reference "#PWR027")
+					(reference "#PWR0100")
 					(unit 1)
 				)
@@
 		(in_pos_files yes)
 		(dnp no)
-		(property "Reference" "U3"
+		(property "Reference" "U12"
 			(at 60.96 30.0482 0)
 			(show_name no)
@@
 			(project "karabas-megasound"
 				(path "/eff1afb7-47ba-46af-a815-4a07fb8d674b/1ef77d13-3c60-4080-9817-a45398794587"
-					(reference "U3")
+					(reference "U12")
 					(unit 1)
 				)
@@
 		(in_pos_files yes)
 		(dnp no)
-		(property "Reference" "#PWR063"
+		(property "Reference" "#PWR0104"
 			(at 81.28 83.82 0)
 			(hide yes)
@@
 			(project "karabas-megasound"
 				(path "/eff1afb7-47ba-46af-a815-4a07fb8d674b/1ef77d13-3c60-4080-9817-a45398794587"
-					(reference "#PWR063")
+					(reference "#PWR0104")
 					(unit 1)
 				)
@@
 		(in_pos_files yes)
 		(dnp no)
-		(property "Reference" "#PWR083"
+		(property "Reference" "#PWR0102"
 			(at 48.26 105.41 0)
 			(hide yes)
@@
 			(project "karabas-megasound"
 				(path "/eff1afb7-47ba-46af-a815-4a07fb8d674b/1ef77d13-3c60-4080-9817-a45398794587"
-					(reference "#PWR083")
+					(reference "#PWR0102")
 					(unit 1)
 				)
@@
 		(in_pos_files yes)
 		(dnp no)
-		(property "Reference" "#PWR031"
+		(property "Reference" "#PWR0103"
 			(at 83.82 105.41 0)
 			(hide yes)
@@
 			(project "karabas-megasound"
 				(path "/eff1afb7-47ba-46af-a815-4a07fb8d674b/1ef77d13-3c60-4080-9817-a45398794587"
-					(reference "#PWR031")
+					(reference "#PWR0103")
 					(unit 1)
 				)
