File: pcb/revA/power.kicad_sch (KiCad schematic)
At the start: 24 parts, among them J5 5V_PRG, U11 1117-1.2, U5 1117-3.3, U6 1117-3.3

Commit message: Initial firmware
Parts:
- renumbered C11 to C40, C21 to C41, C7 to C42, C12 to C43, C22 to C44, C13 to C45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
Other:
- title: karabas-Megasound -> Karabas-MegaBuzz
