File: pcb/revA/vu.kicad_sch (KiCad schematic)
At the start: 32 parts

Commit message: Initial firmware
Parts:
- renumbered D2 to D1, D11 to D10, D12 to D11, D13 to D12, D14 to D13, D15 to D14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
Other:
- title: karabas-Megasound -> Karabas-MegaBuzz
