File: pcb/revA1/audio.kicad_sch (KiCad schematic)
At the start: 43 parts, among them J3 PJ307, J4 Conn_01x04, U10 PCM5102A, U11 PCM1808PWR, U8 YMF262-M, U9 SAM2695

Commit message: revA1, WIP
Parts:
- renumbered C16 to C17, C17 to C18, C18 to C19, C19 to C20, C20 to C21, C21 to C22, C22 to C23, C23 to C24, C24 to C25, C25 to C26, C26 to C29, C29 to C30, C30 to C31, C31 to C32, C32 to C33, C33 to C34, C34 to C35, C35 to C36, C36 to C37, C37 to C38, C38 to C39, J3 to J4, J4 to J5, R13 to R16, R14 to R17, R15 to R18, R16 to R19, R17 to R20, R18 to R21, R19 to R22, R20 to R23, R21 to R24, R22 to R25, R23 to R26, R24 to R27, R25 to R28, R26 to R29, U8 to U10, U9 to U11, U10 to U12, U11 to U13

Commit message: Small improvements to the revA1
Parts:
- added T10, T11, T12, T9: TestPoint2, TestPoint:TestPoint_Pad_D1.5mm, symbol Connector:TestPoint
- J5: now not fitted; now left out of the parts list
Connections:
- net DAC_BCK: now also T9.1
- net DAC_DAT: now also T10.1
- net DAC_WS: now also T11.1
- net GND: now also T12.1
