File: pcb/revA1/karabas-megabuzz.kicad_sch (KiCad schematic)
At the start: 1 part

Commit message: revA1, WIP
Parts:
- renumbered LOGO2 to LOGO1
Other:
- note added: "Buttons"
- note added: "PSRAM"
- note added: "SD"
- note removed: "Button"
Changed lines of the file:
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@@
+	)
+	(rectangle
+		(start 124.46 119.3546)
+		(end 161.29 119.38)
+		(stroke
+			(width 0)
+			(type default)
+		)
+		(fill
+			(type none)
+		)
 	)
 	(rectangle
@@
 	)
 	(rectangle
-		(start 176.53 61.214)
+		(start 177.8 61.214)
 		(end 191.77 66.294)
 		(stroke
@@
 	)
 	(rectangle
+		(start 109.22 116.84)
+		(end 124.46 121.92)
+		(stroke
+			(width 0)
+			(type default)
+		)
+		(fill
+			(type color)
+			(color 255 255 194 1)
+		)
+	)
+	(rectangle
 		(start 214.6046 86.614)
 		(end 214.63 91.694)
@@
 	)
 	(rectangle
+		(start 161.29 115.57)
+		(end 161.3154 119.38)
+		(stroke
+			(width 0)
+			(type default)
+		)
+		(fill
+			(type none)
+		)
+	)
+	(rectangle
 		(start 109.2236 89.0839)
 		(end 124.4636 94.1639)
@@
 	)
 	(rectangle
+		(start 165.2365 61.1529)
+		(end 175.3965 66.2329)
+		(stroke
+			(width 0)
+			(type default)
+		)
+		(fill
+			(type color)
+			(color 255 255 194 1)
+		)
+	)
+	(rectangle
 		(start 109.22 80.01)
 		(end 124.46 85.09)
@@
 	)
 	(rectangle
+		(start 170.1331 66.2858)
+		(end 170.1585 70.0958)
+		(stroke
+			(width 0)
+			(type default)
+		)
+		(fill
+			(type none)
+		)
+	)
+	(rectangle
 		(start 191.77 104.394)
 		(end 207.01 104.4194)
@@
 		)
 	)
-	(text "Button"
+	(text "Buttons"
 		(exclude_from_sim no)
 		(at 113.792 92.71 0)
@@
 		)
 	)
+	(text "SD"
+		(exclude_from_sim no)
+		(at 169.164 64.77 0)
+		(effects
+			(font
+				(size 1.27 1.27)
+			)
+			(justify left bottom)
+		)
+	)
 	(text "Parallel"
 		(exclude_from_sim no)
@@
 		)
 	)
+	(text "QSPI"
+		(exclude_from_sim no)
+		(at 132.08 119.38 0)
+		(effects
+			(font
+				(size 1.27 1.27)
+			)
+			(justify left bottom)
+		)
+	)
 	(text "JTAG"
 		(exclude_from_sim no)
@@
 		(exclude_from_sim no)
 		(at 193.802 106.68 0)
+		(effects
+			(font
+				(size 1.27 1.27)
+			)
+			(justify left bottom)
+		)
+	)
+	(text "PSRAM"
+		(exclude_from_sim no)
+		(at 114.046 120.396 0)
 		(effects
 			(font
@@
 		(in_pos_files yes)
 		(dnp no)
-		(property "Reference" "LOGO2"
+		(property "Reference" "LOGO1"
 			(at 163.83 165.1 0)
 			(hide yes)
@@
 			(project "karabas-megabuzz"
 				(path "/eff1afb7-47ba-46af-a815-4a07fb8d674b"
-					(reference "LOGO2")
+					(reference "LOGO1")
 					(unit 1)
 				)

Commit message: revA1
Parts:
- LOGO1: footprint footprints:andy_karpov_logo4_silk -> footprints:andy_karpov_logo5_silk
Changed lines of the file:
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@@
 	(rectangle
 		(start 214.63 106.68)
-		(end 214.6554 137.16)
+		(end 214.6554 128.27)
 		(stroke
 			(width 0)
@@
 	)
 	(rectangle
-		(start 191.77 137.16)
-		(end 214.63 137.1854)
+		(start 191.77 128.27)
+		(end 214.63 128.2954)
 		(stroke
 			(width 0)
@@
 			)
 		)
-		(property "Footprint" "footprints:andy_karpov_logo4_silk"
+		(property "Footprint" "footprints:andy_karpov_logo5_silk"
 			(at 163.83 175.26 0)
 			(hide yes)
