File: pcb/revA1/memory.kicad_sch (KiCad schematic)
At the start: 2 parts, among them U12 CY62167EV30LL

Commit message: revA1, WIP
Parts:
- added C57: 100n, Capacitor_SMD:C_0603_1608Metric_Pad1.08x0.95mm_HandSolder, symbol Device:C
- added R49: 10k, Resistor_SMD:R_0603_1608Metric_Pad0.98x0.95mm_HandSolder, symbol Device:R
- added U18: APS6404L-3SQRx-SN, Package_SO:SOIC-8_3.9x4.9mm_P1.27mm, symbol Memory_RAM:APS6404L-3SQRx-SN
- renumbered C39 to C40, U12 to U14
Connections:
- net +3V3: now also C57.2, R49.2, U18.8 (VDD)
- net GND: now also C57.1, U18.4 (VSS)
- new net CONF_CLK: U18.6 (SCLK)
- new net CONF_IO0: U18.5 (SI/SIO0)
- new net CONF_IO1: U18.2 (SO/SIO1)
- new net CONF_IO2: U18.3 (SIO2)
- new net CONF_IO3: U18.7 (SIO3)
- new net ~{PSRAM_CS}: R49.1, U18.1 (~{CE})
Other:
- note added: "PSRAM"

Commit message: Small improvements to the revA1
Parts:
- U18: now not fitted; now left out of the parts list
Changed lines of the file:
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@@
 	(title_block
 		(title "Karabas-MegaBuzz")
-		(date "2026-05-27")
+		(date "2026-05-29")
 		(rev "A1")
 		(company "Andy Karpov")
@@
 		(body_style 1)
 		(exclude_from_sim no)
-		(in_bom yes)
+		(in_bom no)
 		(on_board yes)
 		(in_pos_files yes)
-		(dnp no)
+		(dnp yes)
 		(fields_autoplaced yes)
 		(property "Reference" "U18"
