File: pcb/revA1/karabas-megabuzz.kicad_pcb (KiCad board)
At the start: 4 copper layers, 92.2 x 44 mm, 175 parts, among them J1 FPGA JTAG, J2 Conn_02x31_Row_Letter_First, J3 uSD card, J4 PJ307, J5 Conn_01x04, J6 PRG, J7 NMI, SW1 SW_DIP_x05, T1 TestPoint1, T10 TestPoint2, T11 TestPoint2, T12 TestPoint2, T2 TestPoint2, T3 TestPoint, T4 TestPoint, T5 TestPoint, T6 TestPoint, T7 TestPoint, T8 TestPoint, T9 TestPoint2, U1 XC6SLX25-FTG256, U10 YMF262-M, U11 SAM2695, U12 PCM5102A, U13 PCM1808PWR, U14 CY62167EV30LL, U15 1117-3.3, U16 1117-3.3, U17 1117-1.2, U18 APS6404L-3SQRx-SN, U2 W25Q128JVS, U3 74AHCT1G125DB, U4 74AHCT1G125DB, U5 SN74CB3T3245PW, U6 SN74CB3T3245PW, U7 SN74CB3T3245PW, U8 SN74CB3T3245PW, U9 SN74LV1T34DBV, X1 50 MHz

Commit message: Removed polygons under BGA chip on F.Cu layer
Routing:
- net GND: track 123.7 -> 130.0 mm, vias 100 -> 101
Changed lines of the file:
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@@
 		)
 	)
-	(gr_text "M1"
-		(at 179.97 112.92 0)
+	(gr_text "I2S"
+		(at 126.2 118.96 0)
 		(layer "B.SilkS" knockout)
 		(effects
@@
 		)
 	)
-	(gr_text "I2S"
-		(at 126.2 118.96 0)
+	(gr_text "M1"
+		(at 179.97 112.92 0)
 		(layer "B.SilkS" knockout)
 		(effects
@@
 		(start 157.45 115.8)
 		(end 156.489 116.761)
-		(width 0.1)
+		(width 0.2)
 		(layer "F.Cu")
 		(net "GND")
@@
 	)
 	(segment
+		(start 160.45 103.8)
+		(end 161 103.25)
+		(width 0.2)
+		(layer "F.Cu")
+		(net "GND")
+	)
+	(segment
 		(start 158.45 106.8)
 		(end 157.916349 107.333651)
@@
 	)
 	(segment
+		(start 156.218 99.568)
+		(end 156.21 99.568)
+		(width 0.2)
+		(layer "F.Cu")
+		(net "GND")
+	)
+	(segment
+		(start 162.876 102.35)
+		(end 162.888 102.362)
+		(width 0.2)
+		(layer "F.Cu")
+		(net "GND")
+	)
+	(segment
 		(start 169.899901 103.34)
 		(end 169.9 103.34)
@@
 	)
 	(segment
+		(start 161.263603 102.35)
+		(end 162.56 102.35)
+		(width 0.2)
+		(layer "F.Cu")
+		(net "GND")
+	)
+	(segment
 		(start 163.357 125.857)
 		(end 163.576 125.857)
@@
 	)
 	(segment
+		(start 161 102.613603)
+		(end 161.263603 102.35)
+		(width 0.2)
+		(layer "F.Cu")
+		(net "GND")
+	)
+	(segment
 		(start 140.325 123.307)
 		(end 139.7 122.682)
@@
 	)
 	(segment
+		(start 162.888 102.362)
+		(end 163.45 101.8)
+		(width 0.2)
+		(layer "F.Cu")
+		(net "GND")
+	)
+	(segment
 		(start 169.47 112.8)
 		(end 169.94 112.33)
@@
 	)
 	(segment
+		(start 162.814 102.362)
+		(end 162.888 102.362)
+		(width 0.2)
+		(layer "F.Cu")
+		(net "GND")
+	)
+	(segment
 		(start 167.45 102.092893)
 		(end 167.95 102.592893)
@@
 	)
 	(segment
+		(start 162.802 102.35)
+		(end 162.814 102.362)
+		(width 0.2)
+		(layer "F.Cu")
+		(net "GND")
+	)
+	(segment
 		(start 171.439902 110.810098)
 		(end 170.92 111.33)
@@
 		(start 156.489 116.761)
 		(end 156.489 116.84)
-		(width 0.1)
+		(width 0.2)
 		(layer "F.Cu")
 		(net "GND")
@@
 	)
 	(segment
+		(start 162.56 102.35)
+		(end 162.802 102.35)
+		(width 0.2)
+		(layer "F.Cu")
+		(net "GND")
+	)
+	(segment
+		(start 161 103.25)
+		(end 161 102.613603)
+		(width 0.2)
+		(layer "F.Cu")
+		(net "GND")
+	)
+	(segment
 		(start 166.45 114.8)
 		(end 166.93037 114.31963)
@@
 	)
 	(segment
+		(start 157.45 100.8)
+		(end 156.218 99.568)
+		(width 0.2)
+		(layer "F.Cu")
+		(net "GND")
+	)
+	(segment
 		(start 121.33 106.6)
 		(end 124.06 106.6)
@@
 	)
 	(segment
+		(start 162.56 102.35)
+		(end 162.876 102.35)
+		(width 0.2)
+		(layer "F.Cu")
+		(net "GND")
+	)
+	(segment
 		(start 122.15 95.25)
 		(end 124.1 95.25)
@@
 	)
 	(via
+		(at 162.888 102.362)
+		(size 0.45)
+		(drill 0.2)
+		(layers "F.Cu" "B.Cu")
+		(net "GND")
+	)
+	(via
 		(at 152.32 109.57)
 		(size 0.6)
@@
 	)
 	(segment
-		(start 161.640406 102.635)
-		(end 163.020736 102.635)
+		(start 164.340023 100.967023)
+		(end 163.737003 100.364003)
 		(width 0.1)
 		(layer "In2.Cu")
@@
 	)
 	(segment
-		(start 163.737003 100.364003)
-		(end 163.737003 99.949)
+		(start 117.431 98.72)
+		(end 127.569326 98.72)
 		(width 0.1)
 		(layer "In2.Cu")
@@
 	)
 	(segment
-		(start 159.143554 102.28)
-		(end 159.803554 102.94)
+		(start 161.335405 102.94)
+		(end 161.640406 102.635)
+		(width 0.1)
+		(layer "In2.Cu")
+		(net "VU_R0")
+	)
+	(segment
+		(start 141.587447 102.28)
+		(end 159.143554 102.28)
+		(width 0.1)
+		(layer "In2.Cu")
+		(net "VU_R0")
+	)
+	(segment
+		(start 161.640406 102.635)
+		(end 162.559959 102.635)
 		(width 0.1)
 		(layer "In2.Cu")
@@
 	)
 	(segment
-		(start 141.587447 102.28)
-		(end 159.143554 102.28)
+		(start 116.84 98.129)
+		(end 117.431 98.72)
 		(width 0.1)
 		(layer "In2.Cu")
@@
 	)
 	(segment
-		(start 116.84 98.129)
-		(end 117.431 98.72)
+		(start 162.559959 102.635)
+		(end 162.794959 102.87)
 		(width 0.1)
 		(layer "In2.Cu")
@@
 	)
 	(segment
-		(start 163.020736 102.635)
-		(end 164.340023 101.315713)
+		(start 159.143554 102.28)
+		(end 159.803554 102.94)
 		(width 0.1)
 		(layer "In2.Cu")
@@
 	)
 	(segment
-		(start 164.340023 100.967023)
-		(end 163.737003 100.364003)
+		(start 162.794959 102.87)
+		(end 163.068 102.87)
 		(width 0.1)
 		(layer "In2.Cu")
@@
 	)
 	(segment
-		(start 134.371826 105.5225)
-		(end 138.344946 105.5225)
+		(start 159.803554 102.94)
+		(end 161.335405 102.94)
 		(width 0.1)
 		(layer "In2.Cu")
@@
 	)
 	(segment
-		(start 117.431 98.72)
-		(end 127.569326 98.72)
+		(start 134.371826 105.5225)
+		(end 138.344946 105.5225)
 		(width 0.1)
 		(layer "In2.Cu")
@@
 	)
 	(segment
-		(start 161.335405 102.94)
-		(end 161.640406 102.635)
+		(start 164.340023 101.597977)
+		(end 164.340023 100.967023)
 		(width 0.1)
 		(layer "In2.Cu")
@@
 	)
 	(segment
-		(start 164.340023 101.315713)
-		(end 164.340023 100.967023)
+		(start 163.737003 100.364003)
+		(end 163.737003 99.949)
 		(width 0.1)
 		(layer "In2.Cu")
@@
 	)
 	(segment
-		(start 159.803554 102.94)
-		(end 161.335405 102.94)
+		(start 163.068 102.87)
+		(end 164.340023 101.597977)
 		(width 0.1)
 		(layer "In2.Cu")
@@
 	)
 	(segment
-		(start 159.04 102.53)
-		(end 159.7 103.19)
+		(start 161.743959 102.885)
+		(end 162.387578 102.885)
 		(width 0.1)
 		(layer "In2.Cu")
@@
 	)
 	(segment
-		(start 116.292 99.02)
-		(end 127.445062 99.02)
+		(start 138.3985 105.8225)
+		(end 141.691 102.53)
 		(width 0.1)
 		(layer "In2.Cu")
@@
 	)
 	(segment
-		(start 163.195 102.885)
-		(end 164.39 101.69)
+		(start 162.387578 102.885)
+		(end 162.622578 103.12)
 		(width 0.1)
 		(layer "In2.Cu")
@@
 	)
 	(segment
-		(start 159.7 103.19)
-		(end 161.438959 103.19)
+		(start 162.622578 103.12)
+		(end 163.2 103.12)
 		(width 0.1)
 		(layer "In2.Cu")
@@
 	)
 	(segment
-		(start 141.691 102.53)
-		(end 159.04 102.53)
+		(start 161.438958 103.19)
+		(end 161.743959 102.885)
 		(width 0.1)
 		(layer "In2.Cu")
@@
 	)
 	(segment
-		(start 134.247562 105.8225)
-		(end 138.3985 105.8225)
+		(start 163.2 103.12)
+		(end 164.960206 101.359794)
 		(width 0.1)
 		(layer "In2.Cu")
@@
 	)
 	(segment
-		(start 164.960206 101.359794)
-		(end 164.960206 101.300104)
+		(start 114.3 97.028)
+		(end 116.292 99.02)
 		(width 0.1)
 		(layer "In2.Cu")
@@
 	)
 	(segment
-		(start 161.743959 102.885)
-		(end 163.195 102.885)
+		(start 159.04 102.53)
+		(end 159.700001 103.19)
 		(width 0.1)
 		(layer "In2.Cu")
@@
 	)
 	(segment
-		(start 114.3 97.028)
-		(end 116.292 99.02)
+		(start 159.700001 103.19)
+		(end 161.438958 103.19)
 		(width 0.1)
 		(layer "In2.Cu")
@@
 	)
 	(segment
-		(start 138.3985 105.8225)
-		(end 141.691 102.53)
+		(start 134.247562 105.8225)
+		(end 138.3985 105.8225)
 		(width 0.1)
 		(layer "In2.Cu")
@@
 	)
 	(segment
-		(start 161.438959 103.19)
-		(end 161.743959 102.885)
+		(start 141.691 102.53)
+		(end 159.04 102.53)
 		(width 0.1)
 		(layer "In2.Cu")
@@
 	)
 	(segment
-		(start 164.63 101.69)
-		(end 164.960206 101.359794)
+		(start 164.960206 101.359794)
+		(end 164.960206 101.300104)
 		(width 0.1)
 		(layer "In2.Cu")
@@
 	)
 	(segment
-		(start 164.39 101.69)
-		(end 164.63 101.69)
+		(start 116.292 99.02)
+		(end 127.445062 99.02)
 		(width 0.1)
 		(layer "In2.Cu")
@@
 	)
 	(zone
+		(locked yes)
+		(layer "F.Cu")
+		(hatch edge 0.5)
+		(connect_pads
+			(clearance 0)
+		)
+		(min_thickness 0.25)
+		(keepout
+			(tracks allowed)
+			(vias allowed)
+			(pads allowed)
+			(copperpour not_allowed)
+			(footprints allowed)
+		)
+		(placement
+			(enabled no)
+			(sheetname "/")
+		)
+		(fill
+			(thermal_gap 0.5)
+			(thermal_bridge_width 0.5)
+			(island_removal_mode 0)
+		)
+		(polygon
+			(pts
+				(xy 156.718 100.076) (xy 173.228 100.076) (xy 173.228 116.586) (xy 156.718 116.586)
+			)
+		)
+	)
+	(zone

Commit message: Fixed missing LED1 connection, new revA1 release
Parts:
- D1: value L0 -> BLUE
- D10: value R1 -> GREEN
- D11: value R2 -> GREEN
- D12: value R3 -> GREEN
- D13: value R4 -> GREEN
- D14: value R5 -> YELLOW
- D15: value R6 -> YELLOW
- D16: value R7 -> RED
- D17, D8: value L7 -> RED
- D2: value L1 -> GREEN
- D3: value L2 -> GREEN
- D4: value L3 -> GREEN
- D5: value L4 -> GREEN
- D6: value L5 -> YELLOW
- D7: value L6 -> YELLOW
- D9: value R0 -> BLUE
Connections:
- U1 pad D6: unconnected-(U1A-IO_L7P_0-PadD6) -> LED1
Routing:
- net LED1: track 0.00 -> 21.3 mm, vias 0 -> 2
