File: pcb/revB/karabas-megabuzz.kicad_pcb (KiCad board)
At the start: 4 copper layers, 92.2 x 44 mm, 168 parts, among them J1 FPGA JTAG, J2 Conn_02x31_Row_Letter_First, J3 uSD card, J4 PJ307, J5 Conn_01x04, J6 PRG, J7 NMI, SW1 SW_DIP_x05, T1 TestPoint1, T10 TestPoint2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

Commit message: Added revB project files, actual 3d pcb screenshots
Routing:
- net GND: vias 87 -> 88
Other:
- board text added: "Enjoy the buzz :)"
- board text removed: "Enjoy the silence!"
