File: pcb/revB/karabas-megabuzz.kicad_sch (KiCad schematic)
At the start: 1 part

Commit message: Added revB project files, actual 3d pcb screenshots
Other:
- note added: "SDRAM 32MB"
- note removed: "SRAM 2MB"
Changed lines of the file:
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@@
 		)
 	)
-	(text "SRAM\n2MB"
+	(text "SDRAM\n32MB"
 		(exclude_from_sim no)
 		(at 114.3 112.014 0)
