File: pcb/revA2/karabas-megabuzz.kicad_pcb (KiCad board)
At the start: 4 copper layers, 92.2 x 44 mm, 168 parts, among them J1 FPGA JTAG, J2 Conn_02x31_Row_Letter_First, J3 uSD card, J4 PJ307, J5 Conn_01x04, J6 PRG, J7 NMI, T1 TestPoint1, T10 TestPoint2, T11 TestPoint2, T12 TestPoint2, T2 TestPoint2, T3 TestPoint, T4 TestPoint, T5 TestPoint, T6 TestPoint, T7 TestPoint, T8 TestPoint, T9 TestPoint2, U1 XC6SLX25-FTG256, U10 YMF262-M, U11 SAM2695, U12 PCM5102A, U13 PCM1808PWR, U14 CY62167EV30LL, U15 1117-3.3, U16 1117-3.3, U17 1117-1.2, U18 APS6404L-3SQRx-SN, U19 74AHCT1G125DB, U2 W25Q128JVS, U20 AS6C1008-xxST, U21 24LC08, U3 74AHCT1G125DB, U4 74AHCT1G125DB, U5 SN74CB3T3245PW, U6 SN74CB3T3245PW, U7 SN74CB3T3245PW, U8 SN74CB3T3245PW, U9 SN74LV1T34DBV, X1 50 MHz

Commit message: revA2 updates
Parts:
- removed C16: 100n, Capacitor_SMD:C_0603_1608Metric_Pad1.08x0.95mm_HandSolder
- C23, C30: moved to F.Cu
- moved R3 6.91 mm to (157.3, 123.7), turned to -90 degrees
- moved C30 4.93 mm to (122.9, 102.4)
- moved C31 3.75 mm to (120.8, 103.1)
- moved R22 3.51 mm to (125.5, 102.8), turned to -90 degrees
- moved C29 3.16 mm to (124.0, 106.3), turned to -90 degrees
- moved R23 2.97 mm to (124.0, 102.8), turned to -90 degrees
- moved C26 1.83 mm to (125.5, 106.3), turned to -90 degrees
- moved L1 1.71 mm to (117.0, 101.5)
- moved C55 1.33 mm to (120.8, 98.4), turned to 180 degrees
- moved C20 1.30 mm to (125.6, 99.3), turned to -90 degrees
- moved C21 1.27 mm to (124.0, 99.3), turned to -90 degrees
- moved C56 1.13 mm to (116.9, 103.1), turned to 180 degrees
- moved C23 0.76 mm to (127.3, 100.9)
- moved C47 0.64 mm to (155.8, 123.7)
- moved R30 0.62 mm to (125.1, 110.4)
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Routing:
- net MIDI_L: track 15.6 -> 1.72 mm
- net +5V: track 221.8 -> 229.2 mm
- net MIDI_R: track 7.55 -> 1.70 mm
- net Net-(U13-VINL): track 8.77 -> 3.80 mm
- net AGND: track 14.4 -> 19.3 mm
- net +3V3: track 180.9 -> 184.5 mm, vias 51 -> 50
- net GND: track 124.1 -> 127.7 mm, vias 111 -> 115
- net +3V3A: track 47.1 -> 48.8 mm
- net Net-(U13-VREF): track 3.62 -> 2.03 mm
- net Net-(U13-VINR): track 4.15 -> 5.41 mm
- net +1V2: track 43.0 -> 44.2 mm
- net xA12: track 32.1 -> 32.8 mm
- net CONF_PRG_B: track 11.9 -> 11.2 mm
- net +5VA: track 8.66 -> 8.04 mm
- net xA13: track 36.2 -> 36.7 mm
