File: pcb/revA3/audio.kicad_sch (KiCad schematic)
At the start: 43 parts, among them J4 PJ307, J5 Conn_01x04, U10 YMF262-M, U11 SAM2695, U12 PCM5102A, U13 PCM1808PWR, U22 VS1053

Commit message: Updated revA3 with required additional pullups
Parts:
- added R16: 10k, Resistor_SMD:R_0603_1608Metric_Pad0.98x0.95mm_HandSolder, symbol Device:R
- added R17, R18, R19, R29, R56: 100k, Resistor_SMD:R_0603_1608Metric_Pad0.98x0.95mm_HandSolder, symbol Device:R
Connections:
- net +3V3: now also R16.1
- net GND: now also R17.2, R18.2, R19.2, R29.2, R56.2
- net at U22.10 (GPIO3/SDATA): now also U22.11 (GPIO6/I2S_SCLK), U22.12 (GPIO7/I2S_SDATA), U22.9 (GPIO2/DCLK), R56.1
- net at U22.25 (GPIO5/I2S_MCLK): now also R29.1
- net at U22.26 (RX): now also R16.2
- net at U22.33 (GPIO0): now also R17.1
- net at U22.34 (GPIO1): now also R18.1
- net at U22.36 (GPIO4/I2S_LROUT): now also R19.1
- no-connect marks 27 -> 18
