File: pcb/revA3/interfaces.kicad_sch (KiCad schematic)
At the start: 28 parts, among them J2 Conn_02x31_Row_Letter_First, J3 uSD card, J7 NMI, U19 74AHCT1G125DB, U3 74AHCT1G125DB, U4 74AHCT1G125DB, U5 SN74CB3T3245PW, U6 SN74CB3T3245PW, U7 SN74CB3T3245PW, U8 SN74CB3T3245PW, U9 SN74LV1T34DBV

Commit message: Updated revA3 - the reset output on bss138
Parts:
- removed D18: 1N4148W, Diode_SMD:D_SOD-123, symbol Diode:1N4148W
- added Q1: BSS138, Package_TO_SOT_SMD:SOT-23, symbol Transistor_FET:BSS138
- added R57: 10k, Resistor_SMD:R_0603_1608Metric_Pad0.98x0.95mm_HandSolder, symbol Device:R
- R53: value 27 -> 10k
Connections:
- net +3V3: now also R53.1, Q1.1 (G)
- net +5V: now also R57.1
- net ~{RST}: now also Q1.3 (D), R57.2; no longer R53.2
- net ~{oRST}: now also R53.2, Q1.2 (S)
